File: Mir.kicad_pcb (KiCad board)
At the start: 2 copper layers, 265.4 x 111.2 mm, 54 parts, among them SW1 SW_Push, U1 ProMicro

Commit message: Routed
Connections:
- U1 pad 10: Net-(U1-Pad10) -> ROW3
- U1 pad 11: Net-(U1-Pad11) -> ROW4
- U1 pad 12: Net-(U1-Pad12) -> COL3
- U1 pad 13: Net-(U1-Pad13) -> ROW2
- U1 pad 15: Net-(U1-Pad15) -> COL1
- U1 pad 20: Net-(U1-Pad20) -> COL0
- U1 pad 9: Net-(U1-Pad9) -> COL2
Routing:
- net ROW4: track 61.8 -> 115.5 mm
- net ROW3: track 56.7 -> 93.3 mm
- net COL3: track 79.3 -> 112.9 mm
- net COL0: track 80.0 -> 99.4 mm
- net ROW2: track 54.4 -> 73.8 mm
- net COL2: track 78.9 -> 87.5 mm
- net COL1: track 87.9 -> 91.9 mm
Other:
- board text added: "Pro Micro Align the square pads"

Commit message: Add ground fills
Parts:
- removed REF**: outline, locallib:outline
- removed REF** (x8): breakaway-mousebites, random-keyboard-parts:breakaway-mousebites
- added MOUSEBITE1: Mousebites, random-keyboard-parts:breakaway-mousebites, F.Cu at (105.6, 49.2)
- added MOUSEBITE2: Mousebites, random-keyboard-parts:breakaway-mousebites, F.Cu at (108.0, 49.2)
- added MOUSEBITE3: Mousebites, random-keyboard-parts:breakaway-mousebites, F.Cu at (105.6, 106.4)
- added MOUSEBITE4: Mousebites, random-keyboard-parts:breakaway-mousebites, F.Cu at (108.0, 106.4)
- added MOUSEBITE5: Mousebites, random-keyboard-parts:breakaway-mousebites, F.Cu at (28.6, 49.2)
- added MOUSEBITE6: Mousebites, random-keyboard-parts:breakaway-mousebites, F.Cu at (31.0, 49.2)
- added MOUSEBITE7: Mousebites, random-keyboard-parts:breakaway-mousebites, F.Cu at (28.6, 106.4)
- added MOUSEBITE8: Mousebites, random-keyboard-parts:breakaway-mousebites, F.Cu at (31.0, 106.4)
- added O1: Outline, locallib:outline, F.Cu at (200.9, 133.3)
Routing:
- net ROW3: track 93.3 -> 92.6 mm
- net ROW4: track 115.5 -> 114.9 mm
- added copper zone on B.Cu, net Earth
- added copper zone on F.Cu, net Earth
- added copper zone on B.Cu, net GNDA
- added copper zone on F.Cu, net GNDA
