File: Soyuz.kicad_pcb (KiCad board)
At the start: 2 copper layers, 265.4 x 111.2 mm, 54 parts, among them SW1 SW_Push, U1 ProMicro

Commit message: Rename project
Routing:
- net ROW2: track 73.8 -> 72.7 mm
Other:
- board text added: "Numpad kit"
- board text added: "SOYUZ"
Changed lines of the file:
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@@
   (general
     (thickness 1.6)
-    (drawings 11)
+    (drawings 18)
     (tracks 253)
     (zones 0)
@@
     (pad "" np_thru_hole circle (at -2.54 -0.254 270) (size 0.7874 0.7874) (drill 0.7874) (layers *.Cu *.Mask))
   )
+  (gr_line (start 51.59375 123.825) (end 106.3625 39.6875) (layer F.SilkS) (width 1))
+  (gr_line (start 106.3625 37.30625) (end 42.8625 123.825) (layer F.SilkS) (width 0.8))
+  (gr_line (start 33.3375 123.825) (end 106.3625 34.925) (layer F.SilkS) (width 0.6))
+  (gr_line (start 31.75 115.09375) (end 106.3625 32.54375) (layer F.SilkS) (width 0.4))
+  (gr_line (start 31.75 106.3625) (end 106.3625 30.1625) (layer F.SilkS) (width 0.2))
+  (gr_text "Numpad kit" (at 72.23125 63.5 45) (layer F.SilkS)
+    (effects (font (size 1.1 1.1) (thickness 0.2) italic))
+  )
+  (gr_text SOYUZ (at 64.897 69.342 45) (layer F.SilkS)
+    (effects (font (size 3 3) (thickness 0.6) italic))
+  )
   (gr_line (start 65.405 32.639) (end 67.31 32.639) (layer B.SilkS) (width 0.2))
   (gr_line (start 65.405 34.671) (end 65.405 32.639) (layer B.SilkS) (width 0.2))
@@
   (segment (start 79.009 91.059) (end 80.2875 92.3375) (width 0.25) (layer B.Cu) (net 15))
   (segment (start 70.104 91.059) (end 79.009 91.059) (width 0.25) (layer B.Cu) (net 15))
+  (segment (start 95.9 88.9) (end 99.3375 92.3375) (width 0.25) (layer B.Cu) (net 16))
   (segment (start 80.9625 87.3125) (end 89.3445 87.3125) (width 0.25) (layer B.Cu) (net 16))
+  (segment (start 90.932 88.9) (end 95.9 88.9) (width 0.25) (layer B.Cu) (net 16))
   (segment (start 89.3445 87.3125) (end 90.932 88.9) (width 0.25) (layer B.Cu) (net 16))
-  (segment (start 95.9 88.9) (end 99.3375 92.3375) (width 0.25) (layer B.Cu) (net 16))
-  (segment (start 90.932 88.9) (end 95.9 88.9) (width 0.25) (layer B.Cu) (net 16))
   (segment (start 53.18125 106.3625) (end 53.18125 106.26725) (width 0.25) (layer B.Cu) (net 17))
   (segment (start 53.18125 106.26725) (end 51.816 104.902) (width 0.25) (layer B.Cu) (net 17))
@@
   (segment (start 57.023 88.773) (end 55.5625 87.3125) (width 0.25) (layer B.Cu) (net 36))
   (segment (start 63.754 88.773) (end 57.023 88.773) (width 0.25) (layer B.Cu) (net 36))
-  (segment (start 68.2625 81.75625) (end 85.18525 81.75625) (width 0.25) (layer B.Cu) (net 36))
-  (segment (start 90.7415 87.3125) (end 92.3925 87.3125) (width 0.25) (layer B.Cu) (net 36))
-  (segment (start 85.18525 81.75625) (end 90.7415 87.3125) (width 0.25) (layer B.Cu) (net 36))
   (segment (start 49.2125 80.16875) (end 50.06975 80.16875) (width 0.25) (layer F.Cu) (net 36))
   (segment (start 55.5625 85.6615) (end 55.5625 87.3125) (width 0.25) (layer F.Cu) (net 36))
@@
   (segment (start 51.1175 78.26375) (end 49.2125 80.16875) (width 0.25) (layer F.Cu) (net 36))
   (segment (start 51.1175 61.595) (end 51.1175 78.26375) (width 0.25) (layer F.Cu) (net 36))
+  (segment (start 90.297 85.217) (end 92.3925 87.3125) (width 0.25) (layer B.Cu) (net 36))
+  (segment (start 69.215 85.217) (end 90.297 85.217) (width 0.25) (layer B.Cu) (net 36))
+  (segment (start 68.2625 84.2645) (end 69.215 85.217) (width 0.25) (layer B.Cu) (net 36))
   (segment (start 68.2625 100.48875) (end 68.29425 100.48875) (width 0.25) (layer F.Cu) (net 37))
   (segment (start 68.29425 100.48875) (end 70.612 98.171) (width 0.25) (layer F.Cu) (net 37))

Commit message: Create production data
Parts:
- added G***: LOGO, locallib:soyuz-logo-30mm, F.Cu at (61.2, 66.8)
- added G***: LOGO, locallib:ai-4.8-silk, B.Cu at (83.3, 119.9)
- added G***: LOGO, locallib:ai-ring-25mm-mask, B.Cu at (-18.3, 69.8)
Other:
- board text added: "Soyuz Numpad Kit Rev 1.0"
- board text added: "Soyuz PCB R1.0 20190113"
- board text added: "Soyuz by ai03"
- board text added: "This is the bottomside of the plate"
- board text added: "Vendor/Customizing instructions 1. Fork Soyuz on GitHub to create your own copy. Clone onto your PC. 2. Turn your logo into a footprint using bitmap2component, save in locallib.pretty. 3. Place it on the topside of the bottom plate. It is left intentionally blank for this. 4. Alt+3 to render and see if it looks nice. 5. Using the Plot tool, generate the gerbers. The bottom plate is reversible."
- board text added: "kb.ai03.me"
- board text removed: "Numpad kit"
- board text removed: "SOYUZ"

Commit message: Update bottom plate artwork
Parts:
- added G***: LOGO, locallib:soyuz-by-ai03, B.Cu at (-18.3, 92.1)
Other:
- board text added: "Pro Micro Component side faces away"
- board text removed: "Pro Micro Align the square pads"
- board text removed: "Soyuz by ai03"

Commit message: Repair silkscreen
Other:
- board text added: "Pro Micro Component side faces away from PCB"
- board text removed: "Pro Micro Component side faces away"
Changed lines of the file:
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@@
   (gr_line (start 67.31 34.671) (end 65.405 34.671) (layer B.SilkS) (width 0.2))
   (gr_line (start 67.31 32.639) (end 67.31 34.671) (layer B.SilkS) (width 0.2))
-  (gr_text "Pro Micro\n\nComponent side\nfaces away" (at 58.7375 46.83125) (layer B.SilkS)
+  (gr_text "Pro Micro\n\nComponent side\nfaces away\nfrom PCB" (at 58.7375 46.83125) (layer B.SilkS)
     (effects (font (size 1 1) (thickness 0.2)) (justify mirror))
   )
